File: Hardware/Kicad project/ESP32-C3-Low-Power-IoT-Plant-Node.kicad_pcb (KiCad board)
At the start: 4 copper layers, 59.5 x 29.9 mm, 66 parts, among them J1 USB_C_Receptacle_USB2.0_16P, J2 Pump, J3 Soil Sensor, Q1 Q_PMOS_GSD, Q2 Q_NMOS_GSD, SW1 SW_Push, SW2 SW_Push, U1 ESP32-C3, U2 USBLC6-2P6, U3 SHT4x, U4 W25Q16JVSS, U5 TPS61200DRC, U6 MCP73831-2-MC, Y1 40MHz

Commit message: Update hardware design to Rev 2.0
Parts:
- removed D2: SS14, Diode_SMD:D_SMA
- removed REF**: WEEE-Logo_4.2x6mm_SilkScreen, Symbol:WEEE-Logo_4.2x6mm_SilkScreen
- removed REF**: OSHW-Logo_5.7x6mm_SilkScreen, Symbol:OSHW-Logo_5.7x6mm_SilkScreen
- added C23: 1uF, Capacitor_SMD:C_0402_1005Metric, F.Cu at (169.6, 79.0)
- added C24: 1uF, Capacitor_SMD:C_0402_1005Metric, F.Cu at (163.5, 79.0)
- added C25: 1uF, Capacitor_SMD:C_0402_1005Metric, F.Cu at (190.2, 95.3)
- added U8: TLV75733PDBV, Package_TO_SOT_SMD:SOT-23-5, F.Cu at (166.2, 78.8)
- R10: value 562K -> 910K
- R8: value 2M -> 910K
- U6: footprint Package_DFN_QFN:DFN-8-1EP_3x2mm_P0.5mm_EP1.7x1.4mm -> Package_DFN_QFN:DFN-8-1EP_3x2mm_P0.5mm_EP1.75x1.45mm
- moved D1 2.26 mm to (168.4, 90.6)
- moved Q1 1.22 mm to (167.7, 85.1), turned to 0 degrees
- moved G*** 0.85 mm to (180.1, 91.1)
- moved U3 0.85 mm to (188.8, 94.4)
- moved R7 0.48 mm to (169.6, 87.0)
- moved R15 0.20 mm to (190.1, 93.4)
Connections:
- net /AOUT renamed AOUT
- net /BATP renamed BATP
- net /BOOT renamed /03_MCU_Core_System/BOOT
- net /CLK renamed /03_MCU_Core_System/CLK
- net /CS renamed /03_MCU_Core_System/CS
- net /D+ renamed /03_MCU_Core_System/D+
- net /D- renamed /03_MCU_Core_System/D-
- net /DI renamed /03_MCU_Core_System/DI
- net /DO renamed /03_MCU_Core_System/DO
- net /HOLD renamed /03_MCU_Core_System/HOLD
- net /LDR renamed LDR
- net /PUMP renamed PUMP
- net /RESET renamed /03_MCU_Core_System/RESET
- net /SCL renamed SCL
- net /SDA renamed SDA
- net /STAT renamed STAT
- net /USB_D+ renamed USB_D+
- net /USB_D- renamed USB_D-
- net /VDD_SPI renamed /03_MCU_Core_System/VDD_SPI
- net /WP renamed /03_MCU_Core_System/WP
- net /XTAL_N renamed /03_MCU_Core_System/XTAL_N
- net /XTAL_P renamed /03_MCU_Core_System/XTAL_P
- net Net-(U5-L) renamed /02_Power_Management/in_L
- BT1 pad 1: Net-(BT1-+) -> /02_Power_Management/Drain
- C16 pad 1: Net-(BT1-+) -> /02_Power_Management/Drain
- C17 pad 1: Net-(D2-A) -> /02_Power_Management/VIN
- C19 pad 1: +3.3V -> +5V
- D1 pad 1: /VIN -> /02_Power_Management/VIN
- L1 pad 1: /VIN -> /02_Power_Management/VIN
- Q1 pad 2: Net-(BT1-+) -> /02_Power_Management/VIN
- Q1 pad 3: Net-(D2-A) -> /02_Power_Management/Drain
- R10 pad 2: +3.3V -> +5V
- R12 pad 2: Net-(D2-A) -> /02_Power_Management/VIN
- R8 pad 2: Net-(D2-A) -> /02_Power_Management/VIN
- U5 pad 2: +3.3V -> +5V
- U5 pad 5: /VIN -> /02_Power_Management/VIN
- U5 pad 6: /VIN -> /02_Power_Management/VIN
- U6 pad 3: Net-(BT1-+) -> /02_Power_Management/Drain
- U6 pad 4: Net-(BT1-+) -> /02_Power_Management/Drain
Routing:
- net /02_Power_Management/VIN: track 0.00 -> 31.2 mm
- net +5V: track 62.6 -> 89.7 mm, vias 0 -> 3
- net /VIN: track 18.0 -> 0.00 mm
- net Net-(D2-A): track 16.9 -> 0.00 mm
- net Net-(BT1-+): track 13.5 -> 0.00 mm
- net /02_Power_Management/Drain: track 0.00 -> 11.5 mm
- net GND: track 56.8 -> 60.3 mm, vias 194 -> 219
- net +3.3V: track 17.2 -> 16.4 mm
- net PUMP: track 28.3 -> 27.8 mm
Other:
- board text added: "LOW POWER IoT NODE REV 2.0"
- board text removed: "LOW POWER IoT NODE REV 1.0"
