File: Hardware/Kicad project/ESP32-C3-Low-Power-IoT-Plant-Node.kicad_sch (KiCad schematic)
At the start: 63 parts, among them J1 USB_C_Receptacle_USB2.0_16P, J2 Pump, J3 Soil Sensor, Q1 Q_PMOS_GSD, Q2 Q_NMOS_GSD, SW1 SW_Push, SW2 SW_Push, U1 ESP32-C3, U2 USBLC6-2P6, U3 SHT4x, U4 W25Q16JVSS, U5 TPS61200DRC, U6 MCP73831-2-MC, Y1 40MHz

Commit message: Update hardware design to Rev 2.0
Parts:
- removed ANT1: (no value), Custom_RF:RF_TI_Antena_2.4GHz_flipped, symbol Custom_RF:Antenna_Inverted_F
- removed BT1: Battery_Cell, Connector_JST:JST_PH_S2B-PH-K_1x02_P2.00mm_Horizontal, symbol Device:Battery_Cell
- removed C1, C14: 10uF, Capacitor_SMD:C_0402_1005Metric, symbol Device:C
- removed C10, C13, C19, C2, C20, C3, C4, C5, C6, C7: 100nF, Capacitor_SMD:C_0402_1005Metric, symbol Device:C
- removed C11, C12: 10pF, Capacitor_SMD:C_0402_1005Metric, symbol Device:C
- removed C15, C16, C17: 4.7uF, Capacitor_SMD:C_0402_1005Metric, symbol Device:C
- removed C18, C8, C9: 1uF, Capacitor_SMD:C_0402_1005Metric, symbol Device:C
- removed C21, C22: 3.3pF, Capacitor_SMD:C_0402_1005Metric, symbol Device:C
- removed D1, D2, D3: SS14, Diode_SMD:D_SMA, symbol Diode:SS14
- removed FB1: 600R, Resistor_SMD:R_0402_1005Metric, symbol Device:FerriteBead_Small
- removed H1: MountingHole, MountingHole:MountingHole_2.1mm, symbol Mechanical:MountingHole
- removed J1: USB_C_Receptacle_USB2.0_16P, Connector_USB:USB_C_Receptacle_GCT_USB4105-xx-A_16P_TopMnt_Horizontal, symbol Connector:USB_C_Receptacle_USB2.0_16P
- removed J2: Pump, Connector_JST:JST_PH_B2B-PH-K_1x02_P2.00mm_Vertical, symbol Connector:Conn_01x02_Pin
- removed J3: Soil Sensor, Connector_JST:JST_PH_B3B-PH-K_1x03_P2.00mm_Vertical, symbol Connector:Conn_01x03_Pin
- removed L1: 2.2uH, Resistor_SMD:R_0402_1005Metric, symbol Device:L
- removed L2: 2.2nH, Resistor_SMD:R_0402_1005Metric, symbol Device:L
- removed LDR1: LDR07, OptoDevice:R_LDR_5.1x4.3mm_P3.4mm_Vertical, symbol Sensor_Optical:LDR07
- removed Q1: Q_PMOS_GSD, Package_TO_SOT_SMD:SOT-23, symbol Transistor_FET:Q_PMOS_GSD
- removed Q2: Q_NMOS_GSD, Package_TO_SOT_SMD:SOT-23, symbol Transistor_FET:Q_NMOS_GSD
- removed R1, R2: 5.1K, Resistor_SMD:R_0402_1005Metric, symbol Device:R
- removed R10, R12: 562K, Resistor_SMD:R_0402_1005Metric, symbol Device:R
- removed R11: 100K, Resistor_SMD:R_0402_1005Metric, symbol Device:R
- removed R13, R9: 180K, Resistor_SMD:R_0402_1005Metric, symbol Device:R
- removed R14, R17, R3, R4, R5, R6, R7: 10K, Resistor_SMD:R_0402_1005Metric, symbol Device:R
- removed R15, R16: 4.7K, Resistor_SMD:R_0402_1005Metric, symbol Device:R
- removed R8: 2M, Resistor_SMD:R_0402_1005Metric, symbol Device:R
- removed SW1, SW2: SW_Push, Button_Switch_SMD:SW_Push_SPST_NO_Alps_SKRK, symbol Switch:SW_Push
- removed U1: ESP32-C3, Package_DFN_QFN:QFN-32-1EP_5x5mm_P0.5mm_EP3.7x3.7mm, symbol MCU_Espressif:ESP32-C3
- removed U2: USBLC6-2P6, Package_TO_SOT_SMD:SOT-666, symbol Power_Protection:USBLC6-2P6
- removed U3: SHT4x, Sensor_Humidity:Sensirion_DFN-4_1.5x1.5mm_P0.8mm_SHT4x_NoCentralPad, symbol Sensor_Humidity:SHT4x
- removed U4: W25Q16JVSS, Package_SO:SOIC-8_5.3x5.3mm_P1.27mm, symbol Memory_Flash:W25Q16JVSS
- removed U5: TPS61200DRC, Package_SON:Texas_S-PVSON-N10_ThermalVias, symbol Regulator_Switching:TPS61200DRC
- removed U6: MCP73831-2-MC, Package_DFN_QFN:DFN-8-1EP_3x2mm_P0.5mm_EP1.7x1.4mm, symbol Battery_Management:MCP73831-2-MC
- removed Y1: 40MHz, Crystal:Crystal_SMD_3225-4Pin_3.2x2.5mm, symbol Device:Crystal_GND23
Connections:
- no-connect marks 7 -> 0
Other:
- added sheet 02_Power_Management (02_Power_Management.kicad_sch)
- added sheet 03_MCU_Core_System (03_MCU_Core_System.kicad_sch)
- added sheet 04_Peripherals_Sensors (04_Peripherals_Sensors.kicad_sch)
- note added: "+3.3V"
- note added: "+3.3VA (Filtred)"
- note added: "+5V"
- note added: "Analog Core"
- note added: "Digital Core"
- note added: "External Flash Data Logging"
- note added: "GPIO"
- note added: "High-Level System Architecture"
- note added: "I2C"
- note added: "Li-Ion Battery (3.0V - 4.2V)"
- note added: "MCP73831 Charger & Power-Path Switch"
- note added: "MOSFET Driver / Pump 5V Irrigation Load"
- note added: "Moisture Sensor Analog Probe"
- note added: "PWM"
- note added: "Pi-Matching Network (Z = 35 + j10 Ω)"
- note added: "REVISION 2.0 CHANGES * Boost Converter (U1) reconfigured from 3.3V to 5.0V output to support inductive load (Pump). * Updated R10 to 900kΩ / R11 to 100kΩ for 5V feedback loop adjustment. * Corrected UVLO network (R8 changed to 910kΩ) for proper 3.0V battery cutoff protection. * Added dedicated 3.3V LDO regulator down-rail from 5V line to isolate MCU/logic circuitry."
- note added: "Raw VBAT"
- note added: "SHT4x Sensor Temp / Humidity"
- note added: "SPI"
- note added: "TLV75733 3.3V LDO"
- note added: "TPS61200 5V Boost"
- note removed: "2MB FLASH MEMORY"
- note removed: "ANALOG DECOUPLING"
- note removed: "ANALOG FILTRING"
- note removed: "BATTERY VOLTAGE MONITOR"
- note removed: "DIGITAL DECOUPLING"
- note removed: "ESD PROTECTION"
- note removed: "HSE CRYSTAL"
- note removed: "LDR"
- note removed: "LI-ION BATTERY CHARGER"
- note removed: "POWER CIRCUIT BAT/USB"
- note removed: "POWER PATH & 3.3V REGULATION"
- note removed: "PUMP CIRCUIT"
- note removed: "RESET + BOOT CIRCUIT"
- note removed: "RF CIRCUIT"
- note removed: "SOIL SENSOR"
- note removed: "TEMP/HUM SENSOR"
- note removed: "USB-C CIRCUIT"
- note removed: "Z=(35+j10)R"
- note removed: "Z=50R"
